File: Hardware/WingHub.kicad_pcb (KiCad board)
At the start: 2 copper layers, 50.8 x 22.9 mm, 17 parts, among them J1 feather long, J2 feather short, J3 USB_A, SW1 RESET, SW2 DOWNLOADER, U1 CH559T

Commit message: Tracers are updated
Parts:
- moved C2 0.51 mm to (57.7, 42.9)
Routing:
- net /PROG: track 21.3 -> 24.3 mm
- net +3V3: track 39.4 -> 40.2 mm
- net /CS: track 38.9 -> 38.3 mm
- net GND: track 153.2 -> 152.6 mm
Other:
- net class Default: trace_width 0.25 -> 0.3
- net class Voltage: trace_width 0.5 -> 0.3
