File: Hardware/WingHub.sch (KiCad schematic (older format))
At the start: 10 parts, among them J1 feather long, J2 feather short, J3 USB_A, SW1 RESET, SW2 DOWNLOADER, U1 CH559T

Commit message: Firmware folder and WingHub.csv (BOM) created.
Parts:
- C1: Mfr.Part # (none) -> CL21F104ZBCNNNC; Price (none) -> $0.0099; Vendor (none) -> LSCS
- C2: Mfr.Part # (none) -> 0805X335K250CT; Price (none) -> $0.031592; Vendor (none) -> LSCS
- D1: Mfr.Part # (none) -> D-R080508L3-KS2; Price (none) -> $0.015256; Vendor (none) -> LSCS
- J3: Mfr.Part # (none) -> C42643; Price (none) -> $0.0334; Vendor (none) -> LCSC
- R1: Mfr.Part # (none) -> 0805W8J0102T5E; Price (none) -> $0.001866; Vendor (none) -> LSCS
- SW1, SW2: Mfr.Part # (none) -> TS5215A 250gf; Price (none) -> $0.0148; Vendor (none) -> LSCS
- U1: Mfr.Part # (none) -> CH559T; Price (none) -> $1.1231; Vendor (none) -> LSCS
Changed lines of the file:
@@
 F 2 "Package_SO:SSOP-20_5.3x7.2mm_P0.65mm" H 1950 3900 50  0001 C CNN
 F 3 "https://datasheet.lcsc.com/szlcsc/1808111011_WCH-Jiangsu-Qin-Heng-CH559T_C85215.pdf" H 1950 3900 50  0001 C CNN
+F 4 "CH559T" H 1950 3650 50  0001 C CNN "Mfr.Part #"
+F 5 "LSCS" H 1950 3650 50  0001 C CNN "Vendor"
+F 6 "$1.1231" H 1950 3650 50  0001 C CNN "Price"
 	1    1950 3650
 	1    0    0    -1
@@
 F 2 "Capacitor_SMD:C_0805_2012Metric" H 4050 3200 50  0001 C CNN
 F 3 "~" H 4050 3200 50  0001 C CNN
+F 4 "CL21F104ZBCNNNC" H 4050 3200 50  0001 C CNN "Mfr.Part #"
+F 5 "LSCS" H 4050 3200 50  0001 C CNN "Vendor"
+F 6 "$0.0099" H 4050 3200 50  0001 C CNN "Price"
 	1    4050 3200
 	1    0    0    -1
@@
 F 2 "Capacitor_SMD:C_0805_2012Metric" H 3500 3450 50  0001 C CNN
 F 3 "~" H 3500 3450 50  0001 C CNN
+F 4 "0805X335K250CT" H 3500 3450 50  0001 C CNN "Mfr.Part #"
+F 5 "LSCS" H 3500 3450 50  0001 C CNN "Vendor"
+F 6 "$0.031592" H 3500 3450 50  0001 C CNN "Price"
 	1    3500 3450
 	1    0    0    -1
@@
 F 2 "Button_Switch_SMD:SW_SPST_TL3342" H 3350 1400 50  0001 C CNN
 F 3 "~" H 3350 1400 50  0001 C CNN
+F 4 "TS5215A 250gf" H 3350 1200 50  0001 C CNN "Mfr.Part #"
+F 5 "LSCS" H 3350 1200 50  0001 C CNN "Vendor"
+F 6 "$0.0148" H 3350 1200 50  0001 C CNN "Price"
 	1    3350 1200
 	1    0    0    -1
@@
 F 2 "Button_Switch_SMD:SW_SPST_TL3342" H 3350 1850 50  0001 C CNN
 F 3 "~" H 3350 1850 50  0001 C CNN
+F 4 "TS5215A 250gf" H 3350 1650 50  0001 C CNN "Mfr.Part #"
+F 5 "LSCS" H 3350 1650 50  0001 C CNN "Vendor"
+F 6 "$0.0148" H 3350 1650 50  0001 C CNN "Price"
 	1    3350 1650
 	1    0    0    -1
@@
 F 2 "Connector_USB:USB_A_CONNFLY_DS1095-WNR0" H 1525 1350 50  0001 C CNN
 F 3 " ~" H 1525 1350 50  0001 C CNN
+F 4 "C42643" H 1375 1400 50  0001 C CNN "Mfr.Part #"
+F 5 "LCSC" H 1375 1400 50  0001 C CNN "Vendor"
+F 6 "$0.0334" H 1375 1400 50  0001 C CNN "Price"
 	1    1375 1400
 	1    0    0    -1
@@
 F 2 "LED_SMD:LED_0805_2012Metric" H 5250 1375 50  0001 C CNN
 F 3 "~" H 5250 1375 50  0001 C CNN
+F 4 "D-R080508L3-KS2" H 5250 1375 50  0001 C CNN "Mfr.Part #"
+F 5 "LSCS" H 5250 1375 50  0001 C CNN "Vendor"
+F 6 "$0.015256" H 5250 1375 50  0001 C CNN "Price"
 	1    5250 1375
 	1    0    0    -1
@@
 F 2 "Resistor_SMD:R_0805_2012Metric" H 4935 1375 50  0001 C CNN
 F 3 "~" H 4935 1375 50  0001 C CNN
+F 4 "0805W8J0102T5E" V 4935 1375 50  0001 C CNN "Mfr.Part #"
+F 5 "$0.001866" V 4935 1375 50  0001 C CNN "Price"
+F 6 "LSCS" V 4935 1375 50  0001 C CNN "Vendor"
 	1    4935 1375
 	0    1    1    0
